Commit message: rename base_scan frame

File: urdf/brover.urdf (robot description, URDF)
Before this commit: robot brover, 6 links, 5 joints
Links:
- removed link base_scan
- added link base_laser; collision cylinder length=0.0315 radius=0.055; visual cylinder length=0.0315 radius=0.055
Joints:
- joint scan_joint: child base_scan -> base_laser

File: urdf/turtlebro.urdf (robot description, URDF)
Before this commit: robot turtlebro, 6 links, 5 joints
Links:
- removed link base_scan
- added link base_laser; visual cylinder length=0.0515 radius=0.035
Joints:
- joint scan_joint: child base_scan -> base_laser
