Commit message: Add camera to urdf

File: urdf/turtlebro.urdf (robot description, URDF)
Before this commit: robot turtlebro, 6 links, 5 joints
Links:
- added link front_camera; visual box size=0.04 0.04 0.005
- link base_laser: geometry visual cylinder length=0.0615 radius=0.04
- link base_link: geometry visual box size=0.24 0.20 0.05
Joints:
- added joint camera_joint: type fixed, parent base_link, child front_camera, origin xyz=0.06 0 0.055 rpy=0 0.47 0
- joint base_joint: origin xyz=0.0 0.0 0.025 rpy=0 0 0 -> xyz=0.0 0.0 0.035 rpy=0 0 0
- joint scan_joint: origin xyz=0.0 0 0.08 rpy=0 0 3.1415 -> xyz=0.0 0 0.095 rpy=0 0 3.1415
- joint wheel_left_joint: origin xyz=0 0.115 0 rpy=0 0 0 -> xyz=0 0.115 -0.005 rpy=0 0 0
- joint wheel_right_joint: origin xyz=0 -0.115 0 rpy=0 0 0 -> xyz=0 -0.115 -0.005 rpy=0 0 0

Commit message: new lidar and 2 cam model

File: urdf/turtlebro.urdf (robot description, URDF)
Before this commit: robot turtlebro, 7 links, 6 joints
Links:
- added link back_camera; visual box size=0.10 0.01 0.005
Joints:
- added joint back_camera_joint: type fixed, parent base_footprint, child back_camera, origin xyz=-0.12 -0.06 0.25 rpy=-1.57075 0 1.57075
- joint camera_joint: origin xyz=0.06 0 0.055 rpy=0 0.47 0 -> xyz=0.06 0 0.055 rpy=-1.98 0 -1.57075
